File: amiga-floppy-terminator.kicad_sch (KiCad schematic)
At the start: 2 parts, among them J1 Conn_02x17_Odd_Even

Commit message: v02: Invert diode polarity
What I could do wrong, I did.

Both _DCD and _SEL0 are active low, hence the diode must be inverted to
point towards _SEL0.
Connections:
- net _DCD: now also D1.2 (A); no longer D1.1 (K)
- net _SEL0: now also D1.1 (K); no longer D1.2 (A)
Other:
- moved on the sheet: D1
Changed lines of the file:
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@@
 	(symbol
 		(lib_id "Device:D")
-		(at 138.43 76.2 270)
+		(at 138.43 76.2 90)
 		(unit 1)
 		(exclude_from_sim no)
@@
 					(size 1.27 1.27)
 				)
-				(justify left)
+				(justify right)
 			)
 		)
@@
 					(size 1.27 1.27)
 				)
-				(justify left)
+				(justify right)
 			)
 		)
